File: Mainboard-v18.brd (EAGLE design)
At the start: 50 x 50 mm, 37 parts, among them T1 2N3904, T2 2N3904

Commit message: workaround
Connections:
- net GND: now also PAD2.1; no longer PAD3.1
Routing:
- net GND: track 39.2 -> 24.3 mm
Changed lines of the file:
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@@
 <param name="mtCopper" value="0.035mm 0.035mm 0.035mm 0.035mm 0.035mm 0.035mm 0.035mm 0.035mm 0.035mm 0.035mm 0.035mm 0.035mm 0.035mm 0.035mm 0.035mm 0.035mm"/>
 <param name="mtIsolate" value="1.5mm 0.15mm 0.2mm 0.15mm 0.2mm 0.15mm 0.2mm 0.15mm 0.2mm 0.15mm 0.2mm 0.15mm 0.2mm 0.15mm 0.2mm"/>
-<param name="mdWireWire" value="8mil"/>
-<param name="mdWirePad" value="8mil"/>
-<param name="mdWireVia" value="8mil"/>
-<param name="mdPadPad" value="8mil"/>
-<param name="mdPadVia" value="8mil"/>
-<param name="mdViaVia" value="8mil"/>
-<param name="mdSmdPad" value="8mil"/>
-<param name="mdSmdVia" value="8mil"/>
-<param name="mdSmdSmd" value="8mil"/>
+<param name="mdWireWire" value="0.6mm"/>
+<param name="mdWirePad" value="0.6mm"/>
+<param name="mdWireVia" value="0.6mm"/>
+<param name="mdPadPad" value="0.6mm"/>
+<param name="mdPadVia" value="0.6mm"/>
+<param name="mdViaVia" value="0.6mm"/>
+<param name="mdSmdPad" value="0.6mm"/>
+<param name="mdSmdVia" value="0.6mm"/>
+<param name="mdSmdSmd" value="0.6mm"/>
 <param name="mdViaViaSameLayer" value="8mil"/>
 <param name="mnLayersViaInSmd" value="2"/>
@@
 <param name="msMicroVia" value="9.99mm"/>
 <param name="msBlindViaRatio" value="0.5"/>
-<param name="rvPadTop" value="0.25"/>
-<param name="rvPadInner" value="0.25"/>
-<param name="rvPadBottom" value="0.25"/>
+<param name="rvPadTop" value="0.5"/>
+<param name="rvPadInner" value="0.3"/>
+<param name="rvPadBottom" value="0.5"/>
 <param name="rvViaOuter" value="0.25"/>
 <param name="rvViaInner" value="0.25"/>
@@
 <param name="rvMicroViaInner" value="0.25"/>
 <param name="rlMinPadTop" value="12mil"/>
-<param name="rlMaxPadTop" value="20mil"/>
+<param name="rlMaxPadTop" value="45mil"/>
 <param name="rlMinPadInner" value="10mil"/>
-<param name="rlMaxPadInner" value="20mil"/>
+<param name="rlMaxPadInner" value="45mil"/>
 <param name="rlMinPadBottom" value="12mil"/>
-<param name="rlMaxPadBottom" value="20mil"/>
+<param name="rlMaxPadBottom" value="45mil"/>
 <param name="rlMinViaOuter" value="10mil"/>
 <param name="rlMaxViaOuter" value="20mil"/>
@@
 <param name="rlMinMicroViaInner" value="4mil"/>
 <param name="rlMaxMicroViaInner" value="20mil"/>
-<param name="psTop" value="-1"/>
-<param name="psBottom" value="-1"/>
+<param name="psTop" value="1"/>
+<param name="psBottom" value="1"/>
 <param name="psFirst" value="-1"/>
 <param name="psElongationLong" value="100"/>
@@
 <param name="checkFont" value="1"/>
 <param name="checkRestrict" value="1"/>
-<param name="useDiameter" value="13"/>
+<param name="useDiameter" value="15"/>
 <param name="maxErrors" value="50"/>
 </designrules>
@@
 <contactref element="R2" pad="1"/>
 <contactref element="R1" pad="1"/>
-<wire x1="21.5" y1="29.54" x2="31.75" y2="29.54" width="0.4064" layer="16"/>
-<wire x1="43.047321875" y1="40.86035625" x2="31.75" y2="29.54" width="0.4064" layer="16"/>
+<wire x1="21.5" y1="29.54" x2="31.75" y2="29.54" width="0.6096" layer="16"/>
+<wire x1="43.047321875" y1="40.86035625" x2="31.75" y2="29.54" width="0.6096" layer="16"/>
 </signal>
 <signal name="A4">
 <contactref element="U$33" pad="1"/>
 <contactref element="PAD1" pad="1"/>
-<wire x1="38.393790625" y1="44.904753125" x2="33" y2="36.5" width="0.4064" layer="16"/>
-<wire x1="33" y1="36.5" x2="28.5" y2="36.5" width="0.4064" layer="16"/>
+<wire x1="38.393790625" y1="44.904753125" x2="33" y2="36.5" width="0.6096" layer="16"/>
+<wire x1="33" y1="36.5" x2="28.5" y2="36.5" width="0.6096" layer="16"/>
 </signal>
 <signal name="D7">
@@
 <contactref element="LED1" pad="A"/>
 <contactref element="LED2" pad="A"/>
-<wire x1="41.91" y1="24.13" x2="48.12030625" y2="23.584278125" width="0.4064" layer="16"/>
-<wire x1="22.86" y1="13.97" x2="30.48" y2="13.97" width="0.4064" layer="16"/>
-<wire x1="30.48" y1="13.97" x2="32.47" y2="13.97" width="0.4064" layer="16"/>
-<wire x1="32.47" y1="13.97" x2="33" y2="14.5" width="0.4064" layer="16"/>
-<wire x1="33" y1="14.5" x2="41.91" y2="24.13" width="0.4064" layer="16"/>
+<wire x1="41.91" y1="24.13" x2="48.12030625" y2="23.584278125" width="0.6096" layer="16"/>
+<wire x1="22.86" y1="13.97" x2="30.48" y2="13.97" width="0.6096" layer="16"/>
+<wire x1="30.48" y1="13.97" x2="32.47" y2="13.97" width="0.6096" layer="16"/>
+<wire x1="32.47" y1="13.97" x2="33" y2="14.5" width="0.6096" layer="16"/>
+<wire x1="33" y1="14.5" x2="41.91" y2="24.13" width="0.6096" layer="16"/>
 <contactref element="PAD7" pad="1"/>
-<wire x1="22.86" y1="13.97" x2="20.5" y2="14" width="0.4064" layer="16"/>
-<wire x1="20.5" y1="14" x2="12" y2="24" width="0.4064" layer="16"/>
+<wire x1="22.86" y1="13.97" x2="20.5" y2="14" width="0.6096" layer="16"/>
+<wire x1="20.5" y1="14" x2="12" y2="24" width="0.6096" layer="16"/>
 </signal>
 <signal name="N$1">
 <contactref element="T2" pad="1"/>
 <contactref element="LED1" pad="K"/>
-<wire x1="22.86" y1="20.32" x2="22.86" y2="16.51" width="0.4064" layer="16"/>
+<wire x1="22.86" y1="20.32" x2="22.86" y2="16.51" width="0.6096" layer="16"/>
 </signal>
 <signal name="N$2">
 <contactref element="T1" pad="1"/>
 <contactref element="LED2" pad="K"/>
-<wire x1="30.48" y1="16.51" x2="30.48" y2="21.09" width="0.4064" layer="16"/>
+<wire x1="30.48" y1="16.51" x2="30.48" y2="21.09" width="0.6096" layer="16"/>
 </signal>
 <signal name="GND">
 <contactref element="U$30" pad="1"/>
-<contactref element="PAD3" pad="1"/>
 <contactref element="T1" pad="3"/>
 <contactref element="T2" pad="3"/>
@@
 <vertex x="0.67" y="0.67"/>
 </polygon>
-<wire x1="46.4127" y1="35.69755625" x2="48.12030625" y2="29.75571875" width="0.4064" layer="16"/>
+<wire x1="46.4127" y1="35.69755625" x2="48.12030625" y2="29.75571875" width="0.6096" layer="16"/>
 <contactref element="PAD8" pad="1"/>
-<wire x1="24.5" y1="36.5" x2="12" y2="28.5" width="0.4064" layer="16"/>
-<wire x1="48.12030625" y1="29.75571875" x2="39" y2="27.5" width="0.4064" layer="16"/>
+<wire x1="48.12030625" y1="29.75571875" x2="39" y2="27.5" width="0.6096" layer="16"/>
 <wire x1="39" y1="27.5" x2="33.02" y2="21.09" width="0.4064" layer="16"/>
+<contactref element="PAD2" pad="1"/>
 </signal>
 <signal name="N$3">
@@
 <contactref element="T2" pad="2"/>
 <contactref element="R2" pad="2"/>
-<wire x1="21.5" y1="24.46" x2="21.5" y2="22.75" width="0.4064" layer="16"/>
-<wire x1="21.5" y1="22.75" x2="21.59" y2="22.225" width="0.4064" layer="16"/>
+<wire x1="21.5" y1="24.46" x2="21.5" y2="22.75" width="0.6096" layer="16"/>
+<wire x1="21.5" y1="22.75" x2="21.59" y2="22.225" width="0.6096" layer="16"/>
 </signal>
 <signal name="N$5">
 <contactref element="T1" pad="2"/>
 <contactref element="R1" pad="2"/>
-<wire x1="31.75" y1="24.46" x2="31.75" y2="19.185" width="0.4064" layer="16"/>
+<wire x1="31.75" y1="24.46" x2="31.75" y2="19.185" width="0.6096" layer="16"/>
 </signal>
 </signals>
