File: Schematics/Mainboard-v18.brd (EAGLE design)
At the start: 50 x 50 mm, 37 parts, among them T1 2N3904, T2 2N3904

Commit message: To print
Parts:
- removed U$1: LOGO-LPLPA, LilyPad-Wearables:LOGO-LPA
- T1, T2: value 2N3904 -> (none)
Changed lines of the file:
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@@
 <wire x1="12.37" y1="17.48" x2="10.36" y2="21.88" width="0.4064" layer="29" curve="-179.723939"/>
 <wire x1="10.36" y1="21.88" x2="9.67" y2="26.67" width="0.4064" layer="29" curve="-179.846892"/>
-<circle x="26.67" y="26.67" radius="25" width="0.2032" layer="20"/>
+<circle x="26.67" y="26.67" radius="25" width="0.25" layer="20"/>
 <circle x="26.67" y="26.67" radius="25" width="0.1" layer="47"/>
 <circle x="26.67" y="26.67" radius="17" width="0.001" layer="47"/>
@@
 <element name="GND" library="LilyPad-Wearables" package="SEWTAP" value="SEWTAP1" x="5.19" y="29.76" rot="R351.8"/>
 <element name="U$4" library="LilyPad-Wearables" package="SEWTAP" value="SEWTAP1" x="48.15" y="23.58" rot="R171.8"/>
-<element name="U$1" library="LilyPad-Wearables" package="LOGO-LPA" value="LOGO-LPLPA" x="26.67" y="14.97"/>
-<element name="T1" library="transistor" package="TO92" value="2N3904" x="31.75" y="21.09" rot="R180"/>
-<element name="T2" library="transistor" package="TO92" value="2N3904" x="21.59" y="20.32"/>
+<element name="T1" library="transistor" package="TO92" value=" " x="31.75" y="21.09" rot="R180"/>
+<element name="T2" library="transistor" package="TO92" value=" " x="21.59" y="20.32"/>
 <element name="LED1" library="led" package="LED5MM" value="" x="22.86" y="15.24" rot="R90"/>
 <element name="LED2" library="led" package="LED5MM" value="" x="30.48" y="15.24" rot="R90"/>
