File: Schematics/Mainboard-v18.sch (EAGLE design)
At the start: 37 parts, among them T1 2N3904, T2 2N3904

Commit message: To print
Parts:
- removed U$1: LOGO-LPLPA, LilyPad-Wearables:LOGO-LPLPA
- T1, T2: value 2N3904 -> (none)
Changed lines of the file:
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@@
 <part name="P+5" library="SparkFun" deviceset="VCC" device=""/>
 <part name="U$4" library="LilyPad-Wearables" deviceset="SEWTAP" device="1"/>
-<part name="U$1" library="LilyPad-Wearables" deviceset="LOGO-LP" device="LPA"/>
-<part name="T1" library="transistor" deviceset="2N3904" device=""/>
-<part name="T2" library="transistor" deviceset="2N3904" device=""/>
+<part name="T1" library="transistor" deviceset="2N3904" device="" value=" "/>
+<part name="T2" library="transistor" deviceset="2N3904" device="" value=" "/>
 <part name="LED1" library="led" deviceset="LED" device="5MM"/>
 <part name="LED2" library="led" deviceset="LED" device="5MM"/>
@@
 </instance>
 <instance part="U$4" gate="G$1" x="38.1" y="50.8"/>
-<instance part="U$1" gate="G$1" x="236.22" y="17.78"/>
 <instance part="T1" gate="G1" x="99.06" y="154.94"/>
 <instance part="T2" gate="G1" x="76.2" y="154.94"/>
