File: Schematics/LilypadShield(wPower).brd (EAGLE design)
At the start: 50 x 50 mm, 43 parts, among them SW1 RUN, T1 BC850, T2 BC850, U1 NCP1400-5V

Commit message: Shield with smd elements and power supply
Parts:
- moved LED3 12.7 mm to (26.5, 32.8), turned to 180 degrees
- moved R3 11.3 mm to (15.0, 31.2), flipped to the bottom
- moved SW1 8.06 mm to (24.8, 36.0)
- moved C2 4.75 mm to (17.2, 22.0), flipped to the bottom
- moved 100MA 4.50 mm to (17.5, 24.5), flipped to the bottom
- moved D2 2.50 mm to (20.0, 31.5), flipped to the bottom
- moved JP1 2.25 mm to (26.8, 37.8), flipped to the bottom, turned to 180 degrees
- moved D1 2.06 mm to (20.0, 28.0), flipped to the bottom
- moved U1 1.46 mm to (32.0, 30.5), flipped to the bottom
- moved L1 1.03 mm to (26.8, 26.8)
- moved T1 0.75 mm to (31.8, 21.0), turned to 0 degrees
- flipped C10 to the bottom
- flipped C11 to the bottom
- turned R1 to 270 degrees
- turned R2 to 90 degrees
Routing:
- net N$13: track 0.00 -> 46.5 mm, vias 0 -> 4
- net N$12: track 0.00 -> 46.0 mm, vias 0 -> 2
- net B: track 0.00 -> 33.8 mm, vias 0 -> 1
- net A3: track 0.00 -> 33.5 mm, vias 0 -> 2
- net VCC: track 0.00 -> 31.5 mm, vias 0 -> 2
- net C: track 0.00 -> 23.0 mm, vias 0 -> 1
- net N$16: track 0.00 -> 19.9 mm, vias 0 -> 1
- net GND: track 6.18 -> 25.8 mm, vias 0 -> 4
- net N$9: track 0.00 -> 17.5 mm, vias 0 -> 1
- net N$7: track 0.00 -> 14.4 mm
- net N$2: track 0.00 -> 6.86 mm
- net N$5: track 0.00 -> 6.60 mm
- net N$1: track 0.00 -> 6.58 mm
- net N$4: track 0.00 -> 4.83 mm

Commit message: Fixed board
Parts:
- GND, U$30, U$31, U$32, U$33, U$34, U$35, U$36, U$37, U$38, U$39, U$4, U$40, U$41, U$42, U$43, U$44, U$45, U$46, U$47, U$48, U$51: device LilyPad-Wearables:PETAL-LONG-1 -> LilyPad-Wearables:SEWTAP
Connections:
- net VCC: now also U$4.1
Routing:
- net VCC: track 31.5 -> 61.4 mm
- net N$13: track 46.5 -> 58.3 mm
- net GND: track 25.8 -> 36.3 mm
- net N$2: track 6.86 -> 14.4 mm
- net N$12: track 46.0 -> 51.1 mm
- net N$9: track 17.5 -> 22.2 mm
- net A3: track 33.5 -> 36.7 mm, vias 2 -> 6
- net C: track 23.0 -> 26.1 mm
- net N$5: track 6.60 -> 4.81 mm
- net N$16: track 19.9 -> 21.4 mm
- net N$4: track 4.83 -> 4.08 mm
