File: Schematics/LilypadShield(wPower).sch (EAGLE design)
At the start: 43 parts, among them SW1 RUN, T1 BC850, T2 BC850, U1 NCP1400-5V

Commit message: Fixed board
Connections:
- net VCC: now also U$4.1
Changed lines of the file:
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@@
 <classes>
 <class number="0" name="Default" width="0.2032" drill="0">
+<clearance class="0" value="0.355"/>
 </class>
 <class number="1" name="VCC" width="0.3048" drill="0">
+<clearance class="1" value="0.355"/>
 </class>
 </classes>
@@
 <part name="D1" library="SparkFun-Nate" deviceset="DIODE" device="SMA" value="MBRA140"/>
 <part name="P+3" library="SparkFun" deviceset="VCC" device=""/>
+<part name="P+4" library="SparkFun" deviceset="VCC" device=""/>
 </parts>
 <sheets>
@@
 <attribute name="VALUE" x="156.464" y="82.296" size="1.778" layer="96"/>
 </instance>
+<instance part="P+4" gate="1" x="35.56" y="50.8" smashed="yes">
+<attribute name="VALUE" x="34.544" y="54.356" size="1.778" layer="96"/>
+</instance>
 </instances>
 <busses>
@@
 <junction x="157.48" y="78.74"/>
 </segment>
-</net>
+<segment>
+<pinref part="U$4" gate="G$1" pin="1"/>
+<pinref part="P+4" gate="1" pin="VCC"/>
+</segment>
+</net>
