File: Schematics/LilypadShield.brd (EAGLE design)
At the start: 50 x 50 mm, 36 parts, among them T1 , T2 

Commit message: New shields and rename
Parts:
- +: value (none) -> +
- -: value (none) -> -
- renumbered PAD7 to +, PAD8 to -

Commit message: Limiting resistors
Parts:
- added R3, R4: (no value), resistor:0204/5
Connections:
- new net N$6: LED1.A, R3.1
- new net N$7: LED2.A, R4.1
- net VCC: now also R3.2, R4.2; no longer LED1.A, LED2.A
Routing:
- net VCC: track 45.2 -> 53.5 mm
- net N$7: track 0.00 -> 7.15 mm
- net N$6: track 0.00 -> 6.94 mm
Changed lines of the file:
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@@
 <?xml version="1.0" encoding="utf-8"?>
 <!DOCTYPE eagle SYSTEM "eagle.dtd">
-<eagle version="6.4">
+<eagle version="6.5.0">
 <drawing>
 <settings>
@@
 <element name="R1" library="resistor" package="0204/5" value="" x="31.75" y="27" rot="R270"/>
 <element name="R2" library="resistor" package="0204/5" value="" x="21.5" y="27" rot="R270"/>
+<element name="R3" library="resistor" package="0204/5" value="" x="17.5" y="15.25" rot="R270"/>
+<element name="R4" library="resistor" package="0204/5" value="" x="35.5" y="15.25" rot="R270"/>
 </elements>
 <signals>
@@
 <signal name="VCC">
 <contactref element="U$4" pad="1"/>
-<contactref element="LED1" pad="A"/>
-<contactref element="LED2" pad="A"/>
-<wire x1="41.91" y1="24.13" x2="48.12030625" y2="23.584278125" width="0.6096" layer="16"/>
-<wire x1="22.86" y1="13.97" x2="30.48" y2="13.97" width="0.6096" layer="16"/>
-<wire x1="30.48" y1="13.97" x2="32.47" y2="13.97" width="0.6096" layer="16"/>
-<wire x1="32.47" y1="13.97" x2="33" y2="14.5" width="0.6096" layer="16"/>
-<wire x1="33" y1="14.5" x2="41.91" y2="24.13" width="0.6096" layer="16"/>
 <contactref element="+" pad="1"/>
-<wire x1="22.86" y1="13.97" x2="20.5" y2="14" width="0.6096" layer="16"/>
-<wire x1="20.5" y1="14" x2="12" y2="24" width="0.6096" layer="16"/>
+<contactref element="R3" pad="2"/>
+<contactref element="R4" pad="2"/>
+<wire x1="35.5" y1="12.71" x2="35.5" y2="14.5" width="0.4064" layer="16"/>
+<wire x1="35.5" y1="14.5" x2="38.75" y2="17.75" width="0.4064" layer="16"/>
+<wire x1="38.75" y1="17.75" x2="38.75" y2="21" width="0.4064" layer="16"/>
+<wire x1="38.75" y1="21" x2="41.25" y2="23.5" width="0.4064" layer="16"/>
+<wire x1="41.25" y1="23.5" x2="48.036028125" y2="23.5" width="0.4064" layer="16"/>
+<wire x1="48.036028125" y1="23.5" x2="48.12030625" y2="23.584278125" width="0.4064" layer="16"/>
+<wire x1="35.5" y1="12.71" x2="33.46" y2="12.71" width="0.4064" layer="16"/>
+<wire x1="33.46" y1="12.71" x2="31.5" y2="10.75" width="0.4064" layer="16"/>
+<wire x1="31.5" y1="10.75" x2="22" y2="10.75" width="0.4064" layer="16"/>
+<wire x1="22" y1="10.75" x2="19.75" y2="13" width="0.4064" layer="16"/>
+<wire x1="19.75" y1="13" x2="17.79" y2="13" width="0.4064" layer="16"/>
+<wire x1="17.79" y1="13" x2="17.5" y2="12.71" width="0.4064" layer="16"/>
+<wire x1="17.5" y1="12.71" x2="17.5" y2="14.25" width="0.4064" layer="16"/>
+<wire x1="17.5" y1="14.25" x2="16.25" y2="15.5" width="0.4064" layer="16"/>
+<wire x1="16.25" y1="15.5" x2="16.25" y2="16.5" width="0.4064" layer="16"/>
+<wire x1="16.25" y1="16.5" x2="13.75" y2="19" width="0.4064" layer="16"/>
+<wire x1="13.75" y1="19" x2="13.75" y2="22.25" width="0.4064" layer="16"/>
+<wire x1="13.75" y1="22.25" x2="12" y2="24" width="0.4064" layer="16"/>
 </signal>
 <signal name="N$1">
@@
 <wire x1="31.75" y1="22.5" x2="31.75" y2="19.185" width="0.3048" layer="16"/>
 </signal>
+<signal name="N$6">
+<contactref element="LED1" pad="A"/>
+<contactref element="R3" pad="1"/>
+<wire x1="22.86" y1="13.97" x2="22.03" y2="13.97" width="0.4064" layer="16"/>
+<wire x1="22.03" y1="13.97" x2="18.25" y2="17.75" width="0.4064" layer="16"/>
+<wire x1="18.25" y1="17.75" x2="17.54" y2="17.75" width="0.4064" layer="16"/>
+<wire x1="17.54" y1="17.75" x2="17.5" y2="17.79" width="0.4064" layer="16"/>
+</signal>
+<signal name="N$7">
+<contactref element="LED2" pad="A"/>
+<contactref element="R4" pad="1"/>
+<wire x1="30.48" y1="13.97" x2="31.22" y2="13.97" width="0.4064" layer="16"/>
+<wire x1="31.22" y1="13.97" x2="35.75" y2="18.5" width="0.4064" layer="16"/>
+<wire x1="35.75" y1="18.5" x2="35.5" y2="17.79" width="0" layer="19" extent="16-16"/>
+</signal>
 </signals>
