File: Schematics/NanoShield.brd (EAGLE design)
At the start: 17.8 x 43.2 mm, 3 parts, among them J1 HEAD15-NOSS, J2 HEAD15-NOSS-1, SW1 RUN

Commit message: NanoShield
Parts:
- removed SW1: RUN, MySMD:157SW
- added +, -, ., .., ..., ...., B_GND, B_INP: (no value), wirepad:1,6/0,8
- added LED1, LED2, LED3, LED4: (no value), led:LED5MM
- added R1, R2, R3, R4: (no value), resistor:0204/5
- added T1, T2: (no value), transistor:TO92
Connections:
- removed net N$1: J2.4
- new net +5V: J1.4
- new net 3V3: J1.14
- new net N$10: B_INP.1, J2.5
- new net N$3: LED1.K, LED2.K, T1.1
- new net N$4: LED3.K, LED4.K, T2.1
- new net N$5: R1.2, T1.2
- new net N$6: R3.2, T2.2
- new net N$7: LED1.A, LED2.A, R2.1
- new net N$8: LED3.A, LED4.A, R4.1
- new net N$9: J2.6, R1.1, R3.1
- new net VIN: +.1, J1.1, R2.2, R4.2
- net COM: now also -.1, B_GND.1, J1.2, J2.4, J2.7, T1.3, T2.3; no longer J1.4, J2.2
- net N$2: now also J2.1; no longer J2.14
Routing:
- net VIN: track 0.00 -> 49.7 mm
- net N$10: track 0.00 -> 21.8 mm, vias 0 -> 1
- net N$9: track 0.00 -> 19.5 mm
- net N$3: track 0.00 -> 17.6 mm
- net N$4: track 0.00 -> 17.2 mm
- net N$7: track 0.00 -> 8.08 mm
- net N$8: track 0.00 -> 8.03 mm
- net N$5: track 0.00 -> 5.19 mm
- net N$6: track 0.00 -> 5.07 mm
